File: hardware/PCB/klor1_4/klor1_4.kicad_sch (KiCad schematic)
At the start: 68 parts, among them J1 USB_C_Receptacle_USB2.0_16P, SW1 SW_PUSH-MX_W_LED, SW10 SW_PUSH-MX_W_LED, SW11 SW_PUSH-MX_W_LED, SW12 SW_PUSH-MX_W_LED, SW13 SW_PUSH-MX_W_LED, SW14 SW_PUSH-MX_W_LED, SW15 SW_PUSH-MX_W_LED, SW16 SW_PUSH-MX_W_LED, SW17 SW_PUSH-MX_W_LED, SW18 RotaryEncoder_Switch, SW19 SW_PUSH-MX_W_LED, SW2 SW_PUSH-MX_W_LED, SW20 SW_PUSH-MX_W_LED, SW21 SW_PUSH-MX_W_LED, SW22 SW_PUSH-MX_W_LED, SW3 SW_PUSH-MX_W_LED, SW4 SW_PUSH-MX_W_LED, SW5 SW_PUSH-MX_W_LED, SW6 SW_PUSH-MX_W_LED, SW7 SW_PUSH-MX_W_LED, SW8 SW_PUSH-MX_W_LED, SW9 SW_PUSH-MX_W_LED, U1 RP2040-Zero

Commit message: Phase 3e: dual-purpose encoder/MX switch + LED chain integration
Schematic changes:
- Added SW23 (SW_PUSH-MX_W_LED) as dual-purpose alternative to encoder push
- New MX switch shares matrix position [3,5] with encoder push button
  (col5 + SW18B nets, shared diode)
- LED chain extended: SW23B inserted between existing LEDs in chain
- Footprint property fixed: KLOR:SK6812MINI_and_cherry_1 (south-facing variant)

PCB changes:
- SW23 footprint placed at encoder position (overlapping dual-purpose)
- LED chain trace routed (SW23 DOUT -> next LED DIN)
- Encoder MP overlap clearance fixed via repositioning
- GND zone refilled

DRC status: 0 errors, 0 unconnected ✓

Build flexibility: builder choice at assembly
- Install encoder + knob: encoder rotation works (ENCA/ENCB on GP28/GP29)
- Install MX switch + keycap: extra key at matrix [3,5]
- Same PCB design serves both options (no spec change to R1 base 42-key)

Co-Authored-By: Claude Opus 4.7 (1M context) <noreply@anthropic.com>
Parts:
- added SW23: SW_PUSH-MX_W_LED, KLOR:SK6812MINI_and_cherry_1, symbol KLORlib:SW_PUSH-MX_W_LED
Connections:
- net GND: now also SW23.2 (VSS)
- net SW18B: now also SW23.5
- net VCC: now also SW23.4 (VDD)
- net col5: now also SW23.6
- net at JP26.1, SW20.3 (DIN): now also SW23.1 (DOUT); no longer SW19.1 (DOUT)
- new net: SW19.1 (DOUT), SW23.3 (DIN)
Other:
- note added: "USB-C"
- note removed: "TRRS"
- title: Klor Split Keyboard -> KLORID Split Keyboard
- moved on the sheet: JP26, SW10B, SW11B, SW12B, SW13B, SW14B, SW15B, SW16B, SW17B, SW19B, SW1B, SW20B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

Commit message: Phase 3g: add haptic feedback Pimoroni connector (DNP)
Re-add haptic capability dropped in Phase 2, but with DNP flag for
optional install. User decision: V1-only build (no Rev 2 planned), so
add now or skip permanently. Haptic chosen for layering feedback +
curiosity. DNP = order PCB ready, install Pimoroni breakout later.

Schematic:
- Add Conn_01x05_Pin symbol J2 "Haptic_Buzz_DNP" to lib_symbols
- Symbol instance with dnp flag set (red X visual indicator)
- Wire 5 pins in Pimoroni Haptic Buzz pin order: VCC, SDA, SCL,
  HAPTIC_TRIG, GND (direct plug-in via female header, no Dupont)
- I2C SDA/SCL share OLED bus (GP2/GP3, multi-device on same bus)
- HAPTIC_TRIG net new, connected to MCU GP14 (was spare)

PCB:
- Footprint: Connector_PinHeader_2.54mm:PinHeader_1x05_P2.54mm_Vertical
  (5 through-hole pads, 2.54mm pitch, generic header — flexible for
  any DRV2605L breakout sourcing)
- Position: (205.195, 56.44, -90deg) — right half top, near orphan
  silkscreen labels from old fork haptic location (smart placement,
  uses existing labels as visual guide)
- Routed 5 traces to existing nets (VCC, GND, SDA, SCL, HAPTIC_TRIG)

Pin allocation post-haptic: 19 of 20 GPIO used. GP13 = last spare.

Naming correction: HAPTIC_IRQ -> HAPTIC_TRIG (DRV2605L has TRIG input
for external trigger, not IRQ output; Pimoroni labels TRIG; semantically
correct).

DRC: 0 violations, 0 unconnected pads, 0 footprint errors
ERC: 0 errors, 0 warnings (post-rewire 2026-05-18T19:04:53)

Co-Authored-By: Claude Opus 4.7 (1M context) <noreply@anthropic.com>
Parts:
- added J2: Haptic_Buzz_DNP, Connector_PinHeader_2.54mm:PinHeader_1x05_P2.54mm_Vertical, symbol Connector:Conn_01x05_Pin
Connections:
- net GND: now also J2.5 (Pin_5)
- net SCL: now also J2.3 (Pin_3)
- net SDA: now also J2.2 (Pin_2)
- net VCC: now also J2.1 (Pin_1)
- net HAPTIC_TRIG: now reaches U1.9 (GP14)
- net HAPTIC_TRIG: now also J2.4 (Pin_4)
- no-connect marks 6 -> 5
